File: Skyper_Programmer.sch (KiCad schematic (older format))
At the start: 19 parts, among them IC1 LM7805_TO220, IC2 MAX232, IC3 LP2950-3.0_TO92, K1 D-SUB9, K2 1x2, K3 1x4, T1 BC547, T2 BC547

Commit message: Change parts to SMD
Parts:
- removed C6: 10µF, Capacitors_THT:CP_Radial_D5.0mm_P2.00mm, symbol CP
- removed D1: 1N4004, Diodes_THT:D_5W_P5.08mm_Vertical_AnodeUp, symbol D
- removed IC1: LM7805_TO220, TO_SOT_Packages_THT:TO-220-3_Vertical, symbol LM7805_TO220
- removed IC3: LP2950-3.0_TO92, TO_SOT_Packages_THT:TO-92_Inline_Narrow_Oval, symbol LP2950-3.0_TO92
- removed K1: D-SUB9, Connectors_DSub:DSUB-9_Female_Horizontal_Pitch2.77x2.84mm_EdgePinOffset4.94mm_Housed_MountingHolesOffset7.48mm, symbol DB9_Female_MountingHoles
- removed K2: 1x2, Pin_Headers:Pin_Header_Straight_1x02_Pitch2.54mm, symbol Conn_01x02
- removed K3: 1x4, Pin_Headers:Pin_Header_Straight_1x04_Pitch2.54mm, symbol Conn_01x04
- added J1: Pager, Connector_PinHeader_2.54mm:PinHeader_1x04_P2.54mm_Vertical, symbol Connector_Generic:Conn_01x04
- added J10: Pin9, SubD_Connector:SubD Pad, symbol Connector_Generic:Conn_01x01
- added J11: Pin5, SubD_Connector:SubD Pad, symbol Connector_Generic:Conn_01x01
- added J2: USB PWR, Connector_PinSocket_2.54mm:PinSocket_1x02_P2.54mm_Vertical, symbol Connector_Generic:Conn_01x02
- added J3: Pin1, SubD_Connector:SubD Pad, symbol Connector_Generic:Conn_01x01
- added J4: Pin6, SubD_Connector:SubD Pad, symbol Connector_Generic:Conn_01x01
- added J5: Pin2, SubD_Connector:SubD Pad, symbol Connector_Generic:Conn_01x01
- added J6: Pin7, SubD_Connector:SubD Pad, symbol Connector_Generic:Conn_01x01
- added J7: Pin3, SubD_Connector:SubD Pad, symbol Connector_Generic:Conn_01x01
- added J8: Pin8, SubD_Connector:SubD Pad, symbol Connector_Generic:Conn_01x01
- added J9: Pin4, SubD_Connector:SubD Pad, symbol Connector_Generic:Conn_01x01
- added U1: TC1055, Package_TO_SOT_SMD:SOT-23-5, symbol Regulator_Linear:TC1055
- C1: footprint Capacitors_THT:CP_Radial_D5.0mm_P2.00mm -> Capacitors_Tantalum_SMD:CP_Tantalum_Case-A_EIA-3216-18_Reflow; symbol CP -> Skyper_Programmer-rescue:CP
- C2: renamed from C5; footprint Capacitors_THT:CP_Radial_D5.0mm_P2.00mm -> Capacitors_Tantalum_SMD:CP_Tantalum_Case-A_EIA-3216-18_Reflow; symbol CP -> Skyper_Programmer-rescue:CP
- C3: renamed from C2; footprint Capacitors_THT:CP_Radial_D5.0mm_P2.00mm -> Capacitors_Tantalum_SMD:CP_Tantalum_Case-A_EIA-3216-18_Reflow; symbol CP -> Skyper_Programmer-rescue:CP
- C4: renamed from C3; footprint Capacitors_THT:CP_Radial_D8.0mm_P3.80mm -> Capacitors_Tantalum_SMD:CP_Tantalum_Case-A_EIA-3216-18_Reflow; symbol CP -> Skyper_Programmer-rescue:CP
- C5: renamed from C4; footprint Capacitors_THT:CP_Radial_D8.0mm_P3.80mm -> Capacitors_Tantalum_SMD:CP_Tantalum_Case-A_EIA-3216-18_Reflow; symbol CP -> Skyper_Programmer-rescue:CP
- IC1: renamed from IC2; footprint Housings_DIP:DIP-16_W7.62mm -> SMD_Packages:SO-16-N; symbol MAX232-RESCUE-Skyper_Programmer -> Skyper_Programmer-rescue:MAX232-RESCUE-Skyper_Programmer
- R1: renamed from R4; footprint Resistors_THT:R_Axial_DIN0204_L3.6mm_D1.6mm_P7.62mm_Horizontal -> Resistors_SMD:R_0402; symbol R -> Skyper_Programmer-rescue:R
- R2, R3: footprint Resistors_THT:R_Axial_DIN0204_L3.6mm_D1.6mm_P7.62mm_Horizontal -> Resistors_SMD:R_0402; symbol R -> Skyper_Programmer-rescue:R
- R4: renamed from R1; footprint Resistors_THT:R_Axial_DIN0204_L3.6mm_D1.6mm_P7.62mm_Horizontal -> Resistors_SMD:R_0402; symbol R -> Skyper_Programmer-rescue:R
- T1: renamed from T2; value BC547 -> BC847; footprint TO_SOT_Packages_THT:TO-92_Molded_Narrow -> TO_SOT_Packages_SMD:SOT-323_SC-70; symbol BC547 -> Transistor_BJT:BC847
- T2: renamed from T1; value BC547 -> BC847; footprint TO_SOT_Packages_THT:TO-92_Molded_Narrow -> TO_SOT_Packages_SMD:SOT-323_SC-70; symbol BC547 -> Transistor_BJT:BC847
Connections:
- net labels removed: +BATT
- wire segments 63 -> 62
- no-connect marks 0 -> 9
Other:
- note removed: "+9V"
- moved on the sheet: C1
