File: Skyper_Programmer.sch (KiCad schematic (older format))
At the start: 24 parts, among them IC1 MAX232, J1 Pager, J10 Pin9, J11 Pin5, J2 USB PWR, J3 Pin1, J4 Pin6, J5 Pin2, J6 Pin7, J7 Pin3, J8 Pin8, J9 Pin4, T1 BC847, T2 BC847, U1 TC1055

Commit message: Add BOM data
Parts:
- C1: value 10µF -> 10u; MFR (none) -> AVX; MPN (none) -> F931C106KAA; SPN (none) -> 647-F931C106KAA; SPR (none) -> Mouser
- C2, C3, C4, C5: value 1µF -> 1u; MFR (none) -> AVX; MPN (none) -> F931C105MAA; SPN (none) -> 647-F931C105MAA; SPR (none) -> Mouser
- IC1: MFR (none) -> Maxim Integrated; MPN (none) -> MAX232ESE+; SPN (none) -> 700-MAX232ESE; SPR (none) -> Mouser
- R1, R3, R4: MFR (none) -> Panasonic; MPN (none) -> ERJ-PA2F1002X; SPN (none) -> 667-ERJ-PA2F1002X; SPR (none) -> Mouser
- R2: MFR (none) -> Panasonic; MPN (none) -> ERJ-PA2F4702X; SPN (none) -> 667-ERJ-PA2F4702X; SPR (none) -> Mouser
- T1, T2: MFR (none) -> ON Semiconductor; MPN (none) -> SBC847AWT1G; SPN (none) -> 863-SBC847AWT1G; SPR (none) -> Mouser
- U1: MFR (none) -> https://www.mouser.de/datasheet/2/268/21350c-61546.pdf; MPN (none) -> TC1055-3.0VCT713; SPN (none) -> 579-TC1055-3.0VCT713; SPR (none) -> Mouser

Commit message: Change pin header labelling
Other:
- note added: "DSub9 female"
- note added: "EN"
- note added: "RX"
- note added: "TX"
- note removed: "Enable"
- note removed: "Pager IN"
- note removed: "Pager OUT"
